File: rp2040esc.kicad_pcb (KiCad board)
At the start: 2 copper layers, 1.8 x 4.7 mm, 71 parts, among them J101 DRVSEL, J102 BLDC, J103 24VIN, J104 STM32-SWD-POGO, J105 USB_C_2.0, Q101 NCE6020AK, Q102 NCE6020AK, Q103 NCE6020AK, Q104 NCE6020AK, Q105 NCE6020AK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

Commit message: work on layout
Parts:
- C106, C108: footprint Capacitor_THT:CP_Axial_L18.0mm_D10.0mm_P25.00mm_Horizontal -> Capacitor_THT:CP_Radial_D4.0mm_P1.50mm
- moved R103 86.0 mm to (149.9, 109.3)
- moved R105 86.0 mm to (147.0, 109.3)
- moved R107 86.0 mm to (152.9, 109.3)
- moved Q106 85.8 mm to (159.0, 97.5), turned to -90 degrees
- moved Q104 83.8 mm to (150.7, 97.5), turned to -90 degrees
- moved J102 71.8 mm to (159.6, 77.1), turned to 180 degrees
- moved Q103 71.1 mm to (150.8, 85.9), turned to 90 degrees
- moved U101 60.0 mm to (67.7, 103.5)
- moved Q102 53.6 mm to (142.6, 97.5), turned to -90 degrees
- moved Q105 53.5 mm to (159.0, 86.0), turned to 90 degrees
- moved Q101 51.9 mm to (142.6, 85.9), turned to 90 degrees
