File: rp2040esc.kicad_sch (KiCad schematic)
At the start: 70 parts

Commit message: BOM and footprints
Parts:
- removed C?: 10uF, symbol Device:C_Small
- removed C?: 470pF, symbol Device:C_Small
- removed C?: 0.1uF, symbol Device:C_Small
- removed D?: CMS11, symbol Device:D
- removed L?: 4.7uH, symbol Device:L_Small
- removed R?: 3.75k, symbol Device:R_Small_US
- removed R?: 51R, symbol Device:R_Small_US
- removed R?: 1.2k, symbol Device:R_Small_US
- removed U?: R1240, Package_DFN_QFN:DFN-10-1EP_2.6x2.6mm_P0.5mm_EP1.3x2.2mm_ThermalVias, symbol matei:R1240
- added C101: 22uF, Capacitor_SMD:C_1206_3216Metric, symbol Device:C_Small
- added C109: 100nF, Capacitor_SMD:C_0402_1005Metric, symbol Device:C_Small
- added C113: 10uF, Capacitor_SMD:C_0805_2012Metric, symbol Device:C_Small
- added L102: 4.7uH, Inductor_SMD:L_Taiyo-Yuden_NR-30xx, symbol Device:L_Small
- added L103: 20uH, Inductor_SMD:L_1206_3216Metric, symbol Device:L_Small
- added R108: 10k, Resistor_SMD:R_0402_1005Metric, symbol Device:R_Small_US
- added R109: 27k, Resistor_SMD:R_0402_1005Metric, symbol Device:R_Small_US
- added R111: 3.9k, Resistor_SMD:R_0402_1005Metric, symbol Device:R_Small_US
- added TP107: TestPoint, TestPoint:TestPoint_Pad_1.5x1.5mm, symbol Connector:TestPoint
- added U102: RY8310, Package_TO_SOT_SMD:SOT-23-6, symbol matei:RY8310
- C102: renamed from C?; value 47uF -> 22uF; footprint (none) -> Capacitor_SMD:C_1206_3216Metric
- C103, C105, C110, C111, C112, C115, C116, C118: renamed from C?; footprint (none) -> Capacitor_SMD:C_0402_1005Metric
- C104, C107, C114, C117, C119: renamed from C?; footprint (none) -> Capacitor_SMD:C_0805_2012Metric
- C106, C108: renamed from C?; footprint (none) -> Capacitor_THT:CP_Axial_L18.0mm_D10.0mm_P25.00mm_Horizontal; symbol Device:C_Small -> Device:C_Polarized_Small_US
- C120, C121: renamed from C?; value 10uF -> 20pF; footprint (none) -> Capacitor_SMD:C_0402_1005Metric
- D101, D102: renamed from D?; footprint (none) -> Diode_SMD:D_0603_1608Metric
- J101: renamed from J?; footprint (none) -> Jumper:SolderJumper-3_P1.3mm_Open_Pad1.0x1.5mm_NumberLabels
- J102: renamed from J?; footprint (none) -> Connector_JST:JST_XH_S8B-XH-A_1x08_P2.50mm_Horizontal
- J103: renamed from J?; footprint (none) -> Connector_JST:JST_XH_S2B-XH-A_1x02_P2.50mm_Horizontal
- J105: renamed from J?; footprint (none) -> matei:918-418K2022Y40004
- L101: renamed from L?; value 33uH -> 20uH; footprint (none) -> Inductor_SMD:L_1206_3216Metric
- Q101, Q102, Q103, Q104, Q105, Q106: renamed from Q?; value Q_NMOS_DGS -> NCE6020AK; footprint (none) -> Package_TO_SOT_SMD:TO-252-2
- R101, R114, R115, R117: renamed from R?; footprint (none) -> Resistor_SMD:R_0402_1005Metric
- R102, R103, R104, R105, R106, R107: renamed from R?; value 2.2R -> 22; footprint (none) -> Resistor_SMD:R_0402_1005Metric
- R110, R112, R113: renamed from R?; footprint (none) -> Resistor_SMD:R_2512_6332Metric
- R116: renamed from R?; value 100m -> 10k; footprint (none) -> Resistor_SMD:R_0402_1005Metric
- R118, R119: renamed from R?; footprint (none) -> Resistor_SMD:R_0603_1608Metric
- RV101: renamed from RV?; footprint (none) -> Resistor_SMD:R_0402_1005Metric
- SW101: renamed from SW?; footprint (none) -> matei:JS202011JCQN
- SW102: renamed from SW?; footprint (none) -> Resistor_SMD:R_0402_1005Metric
- TP101, TP102, TP103, TP104, TP105, TP106: renamed from TP?; footprint (none) -> TestPoint:TestPoint_Pad_1.5x1.5mm
- U103: renamed from U?; footprint QFN40P700X700X90-57N -> matei:QFN40P700X700X90-57N
- Y101: renamed from Y?; footprint (none) -> Crystal:Crystal_SMD_3225-4Pin_3.2x2.5mm
- gave numbers to parts that had none: 3
Connections:
- net +24V: now also U102.4 (EN), U102.5 (VIN)
- net +3V3: now also C113.1, L102.2, R111.2
- net EXT_IN: now also TP107.1
- net GND: now also C101.1, C113.2, R108.2, U102.2 (GND)
- new net: C109.1, U102.1 (BST)
- new net: R108.1, R109.1, U102.3 (FB)
- new net: C109.2, L102.1, U102.6 (SW)
- new net: R109.2, R111.1
- new net: C101.2, C102.2, L103.1, U101. (nSI)
- new net: L101.1, L103.2
- no-connect marks 5 -> 3
Other:
- moved on the sheet: C102, C107, J103

Commit message: work on layout
Parts:
- C106, C108: footprint Capacitor_THT:CP_Axial_L18.0mm_D10.0mm_P25.00mm_Horizontal -> Capacitor_THT:CP_Radial_D4.0mm_P1.50mm
Changed lines of the file:
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@@
       (effects (font (size 1.27 1.27)) (justify right))
     )
-    (property "Footprint" "Capacitor_THT:CP_Axial_L18.0mm_D10.0mm_P25.00mm_Horizontal" (id 2) (at 96.52 29.21 0)
+    (property "Footprint" "Capacitor_THT:CP_Radial_D4.0mm_P1.50mm" (id 2) (at 96.52 29.21 0)
       (effects (font (size 1.27 1.27)) hide)
     )
@@
       (effects (font (size 1.27 1.27)) (justify right))
     )
-    (property "Footprint" "Capacitor_THT:CP_Axial_L18.0mm_D10.0mm_P25.00mm_Horizontal" (id 2) (at 86.36 29.21 0)
+    (property "Footprint" "Capacitor_THT:CP_Radial_D4.0mm_P1.50mm" (id 2) (at 86.36 29.21 0)
       (effects (font (size 1.27 1.27)) hide)
     )
@@
     )
     (path "/b798a88d-7f0d-4d31-8de8-e577025c154a"
-      (reference "C106") (unit 1) (value "100uF") (footprint "Capacitor_THT:CP_Axial_L18.0mm_D10.0mm_P25.00mm_Horizontal")
+      (reference "C106") (unit 1) (value "100uF") (footprint "Capacitor_THT:CP_Radial_D4.0mm_P1.50mm")
     )
     (path "/7e95ca99-8621-4ba3-8e9a-f909a15ac1df"
@@
     )
     (path "/417aca31-e334-4d08-933f-e3092517f9ed"
-      (reference "C108") (unit 1) (value "100uF") (footprint "Capacitor_THT:CP_Axial_L18.0mm_D10.0mm_P25.00mm_Horizontal")
+      (reference "C108") (unit 1) (value "100uF") (footprint "Capacitor_THT:CP_Radial_D4.0mm_P1.50mm")
     )
     (path "/9e13bf6c-b3be-419f-b00c-b8af50aea318"
